File: pico-1v.kicad_sch (KiCad schematic)
At the start: 49 parts, among them J10 GND, J2 USB-C-2.0, J3 Header-1, J4 Header-2, J5 SWD, J6 USB_B_Micro, J7 VBUS, J8 DM, J9 DP, SW1 UK-B0273-SP25Y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

Commit message: More improvements to schematic
Parts:
- removed J10: GND, CIRCUITSTATE_Pads:Solderpad_Rectangle_0.8x1.3mm_Chamfered, symbol Connector_Generic:Conn_01x01
- removed J7: VBUS, CIRCUITSTATE_Pads:Solderpad_Rounded_Rectangle_0.8x1.3mm, symbol Connector_Generic:Conn_01x01
- removed J8: DM, CIRCUITSTATE_Pads:Solderpad_Rounded_Rectangle_0.8x1.3mm, symbol Connector_Generic:Conn_01x01
- removed J9: DP, CIRCUITSTATE_Pads:Solderpad_Rounded_Rectangle_0.8x1.3mm, symbol Connector_Generic:Conn_01x01
- C1, C13, C14, C15, C16, C17: footprint (none) -> Capacitor_SMD:C_0402_1005Metric
- J2: footprint CIRCUITSTATE_Connector_USB:USB_C_Receptacle_HRO_TYPE-C-31-M-12 -> ExtraFootprints:USB_C_RECEPTACLE_31_M_12
- J3, J4: footprint CIRCUITSTATE-Connector-Pin-Headers:PinHeader_1x20_2H_P2.54mm_Vertical -> Connector_PinHeader_2.54mm:PinHeader_1x20_P2.54mm_Vertical
- R1, R2: footprint (none) -> Resistor_SMD:R_0201_0603Metric
- SW1: footprint CIRCUITSTATE_Switch_SMD:CK_SW_SPST_UK-B0273-SP25Y -> Button_Switch_SMD:SW_Push_1P1T_NO_CK_KMR2
- SW2: footprint (none) -> Button_Switch_SMD:SW_Push_1P1T_NO_CK_KMR2
- SW4: footprint (none) -> Button_Switch_THT:SW_CK_JS202011CQN_DPDT_Straight
- U1: footprint CIRCUITSTATE-QFN:RP2040-QFN-56 -> Package_DFN_QFN:QFN-56-1EP_7x7mm_P0.4mm_EP3.2x3.2mm; symbol CIRCUITSTATE-Microcontrollers:RP2040 -> MCU_RaspberryPi:RP2040
Other:
- moved on the sheet: R5, R6
