File: pico-1v.kicad_sch (KiCad schematic)
At the start: 45 parts, among them J2 USB-C-2.0, J3 Header-1, J4 Header-2, J5 SWD, J6 USB_B_Micro, SW1 UK-B0273-SP25Y, SW2 USB Boot, SW4 SW_Slide_DPDT, U1 RP2040, U2 NCP1117-1.8_SOT223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

Commit message: Updated some stuff
Parts:
- Y1: footprint (none) -> Oscillator:Oscillator_SMD_Abracon_ASE-4Pin_3.2x2.5mm
Connections:
- net GND: now also Y1.2 (GND); no longer Y1. (GND)
Changed lines of the file:
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@@
 			)
 		)
-		(property "Footprint" ""
+		(property "Footprint" "Oscillator:Oscillator_SMD_Abracon_ASE-4Pin_3.2x2.5mm"
 			(at 104.14 187.96 0)
 			(effects
@@
 		(pin "1"
 		)
-		(pin ""
+		(pin "2"
 		)
 		(pin "4"

Commit message: PCB
Parts:
- removed J6: USB_B_Micro, Connector_USB:USB_Micro-B_Molex-105017-0001, symbol Connector:USB_B_Micro
- removed U2: NCP1117-1.8_SOT223, Package_TO_SOT_SMD:SOT-223-3_TabPin2, symbol Regulator_Linear:NCP1117-1.8_SOT223
- removed U3: NCP1117-3.3_SOT223, Package_TO_SOT_SMD:SOT-223-3_TabPin2, symbol Regulator_Linear:NCP1117-3.3_SOT223
- added U2: MCP1703Ax-180xxTT, Package_TO_SOT_SMD:SOT-23, symbol Regulator_Linear:MCP1703Ax-180xxTT
- added U3: MCP1703Ax-330xxTT, Package_TO_SOT_SMD:SOT-23, symbol Regulator_Linear:MCP1703Ax-330xxTT
- Y1: footprint Oscillator:Oscillator_SMD_Abracon_ASE-4Pin_3.2x2.5mm -> ExtraFootprints:ECS-3225MV-120-BN-TR3
Connections:
- net +1V8: now also U2.2 (VO)
- net +3V3: now also U3.2 (VO); no longer C10.1, C11.1, C12.1, C5.1, C6.1, C7.1, C8.1, C9.1
- net GND: now also C1.2, U2.1 (GND), U3.1 (GND)
- net VDD: now also C10.1, C11.1, C12.1, C5.1, C6.1, C7.1, C8.1, C9.1
- net VSYS: now also U2.3 (VI), U3.3 (VI)
- net GPIO23: no longer names the net of U1.35 (GPIO23)
- net GPIO24: no longer names the net of U1.36 (GPIO24)
- net GPIO25: no longer names the net of U1.37 (GPIO25)
- no-connect marks 5 -> 7
Other:
- note removed: "Pads should be masked out if not using Micro-USB. Otherwise, USB-C connector will cause a short."
- note removed: "USB-MICRO"
- moved on the sheet: C19, D3, R8, R9, SW1

Commit message: Rev 1 PCB
Parts:
- H1, H2, H3, H4: footprint MountingHole:MountingHole_2.2mm_M2 -> MountingHole:MountingHole_2.1mm
Changed lines of the file:
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@@
 	)
 	(global_label "USB_D+"
-		(shape input)
+		(shape bidirectional)
 		(at 36.83 67.31 180)
 		(fields_autoplaced yes)
@@
 		)
 		(property "Intersheetrefs" "${INTERSHEET_REFS}"
-			(at 26.1297 67.31 0)
+			(at 25.1137 67.31 0)
 			(effects
 				(font
@@
 	)
 	(global_label "USB_D-"
-		(shape output)
+		(shape bidirectional)
 		(at 274.32 110.49 0)
 		(fields_autoplaced yes)
@@
 		)
 		(property "Intersheetrefs" "${INTERSHEET_REFS}"
-			(at 285.0203 110.49 0)
+			(at 286.0363 110.49 0)
 			(effects
 				(font
@@
 	)
 	(global_label "USB_D+"
-		(shape output)
+		(shape bidirectional)
 		(at 274.32 115.57 0)
 		(fields_autoplaced yes)
@@
 		)
 		(property "Intersheetrefs" "${INTERSHEET_REFS}"
-			(at 285.0203 115.57 0)
+			(at 286.0363 115.57 0)
 			(effects
 				(font
@@
 	)
 	(global_label "USB_D-"
-		(shape input)
+		(shape bidirectional)
 		(at 36.83 69.85 180)
 		(fields_autoplaced yes)
@@
 		)
 		(property "Intersheetrefs" "${INTERSHEET_REFS}"
-			(at 26.1297 69.85 0)
+			(at 25.1137 69.85 0)
 			(effects
 				(font
@@
 			)
 		)
-		(property "Footprint" "MountingHole:MountingHole_2.2mm_M2"
+		(property "Footprint" "MountingHole:MountingHole_2.1mm"
 			(at 38.354 189.23 0)
 			(effects
@@
 			)
 		)
-		(property "Footprint" "MountingHole:MountingHole_2.2mm_M2"
+		(property "Footprint" "MountingHole:MountingHole_2.1mm"
 			(at 38.354 179.07 0)
 			(effects
@@
 			)
 		)
-		(property "Footprint" "MountingHole:MountingHole_2.2mm_M2"
+		(property "Footprint" "MountingHole:MountingHole_2.1mm"
 			(at 38.354 194.31 0)
 			(effects
@@
 			)
 		)
-		(property "Footprint" "MountingHole:MountingHole_2.2mm_M2"
+		(property "Footprint" "MountingHole:MountingHole_2.1mm"
 			(at 38.354 184.15 0)
 			(effects

Commit message: More stuff
Parts:
- C1, C17: value 100n -> 0.1uF
- C13, C14, C15, C16: value 10u -> 10uF
Changed lines of the file:
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@@
 			)
 		)
-		(property "Value" "100n"
+		(property "Value" "0.1uF"
 			(at 386.08 46.9899 0)
 			(effects
@@
 		(on_board yes)
 		(dnp no)
-		(fields_autoplaced yes)
 		(property "Reference" "U4"
-			(at 379.73 52.0699 0)
+			(at 376.428 65.532 0)
 			(effects
 				(font
@@
 		)
 		(property "Value" "AT25FF161A-SSHN-T"
-			(at 379.73 54.6099 0)
+			(at 347.726 41.148 0)
 			(effects
 				(font
@@
 			)
 		)
-		(property "Value" "10u"
+		(property "Value" "10uF"
 			(at 325.12 120.6499 0)
 			(effects
@@
 			)
 		)
-		(property "Value" "100n"
+		(property "Value" "0.1uF"
 			(at 91.44 185.4199 0)
 			(effects
@@
 			)
 		)
-		(property "Value" "10u"
+		(property "Value" "10uF"
 			(at 396.24 120.6499 0)
 			(effects
@@
 			)
 		)
-		(property "Value" "10u"
+		(property "Value" "10uF"
 			(at 368.3 120.6499 0)
 			(effects
@@
 			)
 		)
-		(property "Value" "10u"
+		(property "Value" "10uF"
 			(at 353.06 120.6499 0)
 			(effects

Commit message: Various fixes
Parts:
- removed H1, H2, H3, H4: MountingHole, MountingHole:MountingHole_2.1mm, symbol Mechanical:MountingHole
- removed J5: SWD, Connector_PinHeader_2.54mm:PinHeader_1x03_P2.54mm_Vertical, symbol Connector_Generic:Conn_01x03
- removed SW4: SW_Slide_DPDT, Button_Switch_THT:SW_CK_JS202011CQN_DPDT_Straight, symbol Switch:SW_Slide_DPDT
- added C18: C, Capacitor_SMD:C_0402_1005Metric, symbol Device:C
- added J2: VOLTSEL, Connector_PinHeader_2.54mm:PinHeader_1x03_P2.54mm_Vertical, symbol Connector_Generic:Conn_01x03
- added J5: Conn_02x05_Odd_Even, Connector_PinHeader_1.27mm:PinHeader_2x05_P1.27mm_Vertical_SMD, symbol Connector_Generic:Conn_02x05_Odd_Even
- added R10, R11: 10k, Resistor_SMD:R_0402_1005Metric, symbol Device:R_Small
- added R9: 1k, Resistor_SMD:R_0402_1005Metric, symbol Device:R_Small
- added U5: LMV331, Package_TO_SOT_SMD:SOT-353_SC-70-5, symbol Comparator:LMV331
- R1, R2: footprint Resistor_SMD:R_0201_0603Metric -> Resistor_SMD:R_0402_1005Metric
- renumbered J2 to J1, R8 to R7, R9 to R8
Connections:
- net AREF is gone; now on net +3V3: J4.6 (Pin_6)
- net +1V8: now also J2.3 (Pin_3)
- net +3V3: now also C18.1, J2.1 (Pin_1), R9.2, U5.5 (V+)
- net GND: now also C18.2, J5.3 (Pin_3), J5.5 (Pin_5), J5.9 (Pin_9), R10.1, U5.2 (V-)
- net SWCLK: now also J5.4 (Pin_4)
- net SWDIO: now also J5.2 (Pin_2)
- net VDD: now also J2.2 (Pin_2), J5.1 (Pin_1), R11.1, U5.1 (+)
- net VOLTAGE_MODE: now also R11.2, U5.4
- net USB_DM: now reaches R6.2, U1.46 (USB_DM)
- net USB_DP: now reaches R5.2, U1.47 (USB_DP)
- net V_EN: no longer names the net of J4.4 (Pin_4)
- new net: R10.2, R9.1, U5.3 (-)
- no-connect marks 7 -> 12
Other:
- note removed: "MOUNTING HOLES"
- moved on the sheet: C10, C11, C12, C2, C3, C4, C5, C6, C7, C8, C9, D3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
